Commit message: Start tuning physical pushing system

File: models/pusher.xacro (robot description, xacro)
@@ -1,5 +1,5 @@
 <?xml version="1.0"?>
 <robot xmlns:xacro="http://www.ros.org/wiki/xacro" name="pusher">
-<xacro:property name="m" value="10.02" />
+<xacro:property name="m" value="1.0" />
 <xacro:property name="l" value="0.15" />
 <xacro:property name="r" value="0.02" />

File: pusher.urdf (robot description, URDF)
Before this commit: robot pusher, 1 links, 0 joints
Links:
- link base_link: mass 6.0 -> 1.0
