Commit message: Increase spinning friction to prevent long drifts

File: models/block_big.xacro (robot description, xacro)
@@ -1,5 +1,5 @@
 <?xml version="1.0"?>
 <robot xmlns:xacro="http://www.ros.org/wiki/xacro" name="block_big">
-<xacro:property name="m" value="10.02" />
+<xacro:property name="m" value="2.0" />
 <xacro:property name="l" value="0.15" />
 <xacro:property name="w" value="0.15" />
@@ -7,6 +7,6 @@
   <link name="base_link">
     <contact>
-      <lateral_friction value="2.5"/>
-      <spinning_friction value=".01"/>
+      <lateral_friction value="1.5"/>
+      <spinning_friction value=".5"/>
     </contact>
     <inertial>
@@ -21,5 +21,5 @@
       </geometry>
       <material name="blockmat">
-        <color rgba="0.1 0.7 0.1 1"/>
+        <color rgba="0.1 0.7 0.1 0.8"/>
       </material>
     </visual>

Commit message: Reduce turning friction to make turning easier

File: models/block_big.xacro (robot description, xacro)
@@ -1,5 +1,5 @@
 <?xml version="1.0"?>
 <robot xmlns:xacro="http://www.ros.org/wiki/xacro" name="block_big">
-<xacro:property name="m" value="6.0" />
+<xacro:property name="m" value="3.0" />
 <xacro:property name="l" value="0.35" />
 <xacro:property name="w" value="0.35" />
@@ -11,6 +11,6 @@
     <contact>
       <lateral_friction value="0.8"/>
-      <spinning_friction value=".1"/>
-      <rolling_friction value=".1"/>
+      <spinning_friction value=".05"/>
+      <rolling_friction value=".01"/>
     </contact>
     <inertial>

File: models/pusher.xacro (robot description, xacro)
@@ -6,5 +6,5 @@
   <link name="base_link">
     <contact>
-      <lateral_friction value="1.0"/>
+      <lateral_friction value="1.5"/>
       <spinning_friction value=".1"/>
     </contact>

File: models/wall.xacro (robot description, xacro)
@@ -10,5 +10,5 @@
   <link name="base_link">
     <contact>
-      <lateral_friction value="1.0"/>
+      <lateral_friction value="0.5"/>
       <spinning_friction value=".001"/>
     </contact>
@@ -24,5 +24,5 @@
       </geometry>
       <material name="blockmat">
-        <color rgba="0.2 0.1 0.2 1"/>
+        <color rgba="0.5 0.5 0.5 0.8"/>
       </material>
     </visual>
