Commit message: Create short wall urdf

File: models/short_wall.xacro (robot description, xacro)
@@ -2,4 +2,4 @@
 <robot xmlns:xacro="http://www.ros.org/wiki/xacro" name="wall">
 <xacro:include filename="_wall_base.xacro"/>
-<wall l="3" w="0.5" h="0.3"/>
+<wall l="1.5" w="0.5" h="0.3"/>
 </robot>

File: short_wall.urdf (robot description, URDF)
Before this commit: robot wall, 1 links, 0 joints
Links:
- link base_link: geometry collision box size=1.5 0.5 0.3; visual box size=1.5 0.5 0.3
