Commit message: Use new pusher and block models with better frictional interactions

File: block_big.urdf (robot description, URDF)
Before this commit: robot block_big, 1 links, 0 joints
Links:
- link base_link: mass 2.0 -> 6.0

Commit message: Reduce block height to avoid tipping over and make xacro consistent with current URDF

File: block_big.urdf (robot description, URDF)
Before this commit: robot block_big, 1 links, 0 joints
Links:
- link base_link: geometry collision box size=0.15 0.15 0.15; visual box size=0.15 0.15 0.05

File: models/block_big.xacro (robot description, xacro)
@@ -1,12 +1,12 @@
 <?xml version="1.0"?>
 <robot xmlns:xacro="http://www.ros.org/wiki/xacro" name="block_big">
-<xacro:property name="m" value="2.0" />
+<xacro:property name="m" value="6.0" />
 <xacro:property name="l" value="0.15" />
 <xacro:property name="w" value="0.15" />
-<xacro:property name="h" value="0.15" />
+<xacro:property name="h" value="0.05" />
   <link name="base_link">
     <contact>
       <lateral_friction value="0.8"/>
-      <spinning_friction value=".5"/>
+      <spinning_friction value=".07"/>
     </contact>
     <inertial>

File: models/pusher.xacro (robot description, xacro)
@@ -6,6 +6,6 @@
   <link name="base_link">
     <contact>
-      <lateral_friction value="0.5"/>
-      <spinning_friction value=".01"/>
+      <lateral_friction value="1.0"/>
+      <spinning_friction value=".1"/>
     </contact>
     <inertial>

Commit message: Increase block size

File: block_big.urdf (robot description, URDF)
Before this commit: robot block_big, 1 links, 0 joints
Links:
- link base_link: geometry collision box size=0.55 0.55 0.05; visual box size=0.55 0.55 0.05

File: models/block_big.xacro (robot description, xacro)
@@ -2,16 +2,20 @@
 <robot xmlns:xacro="http://www.ros.org/wiki/xacro" name="block_big">
 <xacro:property name="m" value="6.0" />
-<xacro:property name="l" value="0.15" />
-<xacro:property name="w" value="0.15" />
+<xacro:property name="l" value="0.55" />
+<xacro:property name="w" value="0.55" />
 <xacro:property name="h" value="0.05" />
+<xacro:property name="Ih" value="${1/12*m*(w*w + l*l)}" />
+<xacro:property name="Iw" value="${1/12*m*(h*h + l*l)}" />
+<xacro:property name="Il" value="${1/12*m*(w*w + h*h)}" />
   <link name="base_link">
     <contact>
-      <lateral_friction value="0.8"/>
-      <spinning_friction value=".07"/>
+      <lateral_friction value="0.9"/>
+      <spinning_friction value=".1"/>
+      <rolling_friction value=".1"/>
     </contact>
     <inertial>
       <origin rpy="0 0 0" xyz="0 0 0"/>
       <mass value="${m}"/>
-      <inertia ixx="1" ixy="0" ixz="0" iyy="1" iyz="0" izz="1"/>
+      <inertia ixx="${Il}" ixy="0" ixz="0" iyy="${Iw}" iyz="0" izz="${Ih}"/>
     </inertial>
     <visual>

Commit message: Adjust parameters to get 5-6% rotational error

File: block_big.urdf (robot description, URDF)
Before this commit: robot block_big, 1 links, 0 joints
Links:
- link base_link: geometry collision box size=0.35 0.35 0.05; visual box size=0.35 0.35 0.05

File: models/block_big.xacro (robot description, xacro)
@@ -2,6 +2,6 @@
 <robot xmlns:xacro="http://www.ros.org/wiki/xacro" name="block_big">
 <xacro:property name="m" value="6.0" />
-<xacro:property name="l" value="0.55" />
-<xacro:property name="w" value="0.55" />
+<xacro:property name="l" value="0.35" />
+<xacro:property name="w" value="0.35" />
 <xacro:property name="h" value="0.05" />
 <xacro:property name="Ih" value="${1/12*m*(w*w + l*l)}" />
@@ -10,5 +10,5 @@
   <link name="base_link">
     <contact>
-      <lateral_friction value="0.9"/>
+      <lateral_friction value="0.8"/>
       <spinning_friction value=".1"/>
       <rolling_friction value=".1"/>

Commit message: Tune physical pusher to complete tasks fast enough

File: block_big.urdf (robot description, URDF)
Before this commit: robot block_big, 1 links, 0 joints
Links:
- link base_link: mass 6.0 -> 3.0

Commit message: Make block smaller to make it relatively easier to rotate

File: block_big.urdf (robot description, URDF)
Before this commit: robot block_big, 1 links, 0 joints
Links:
- link base_link: geometry collision box size=0.3 0.3 0.05; visual box size=0.3 0.3 0.05

File: models/block_big.xacro (robot description, xacro)
@@ -2,6 +2,6 @@
 <robot xmlns:xacro="http://www.ros.org/wiki/xacro" name="block_big">
 <xacro:property name="m" value="3.0" />
-<xacro:property name="l" value="0.35" />
-<xacro:property name="w" value="0.35" />
+<xacro:property name="l" value="0.30" />
+<xacro:property name="w" value="0.30" />
 <xacro:property name="h" value="0.05" />
 <xacro:property name="Ih" value="${1/12*m*(w*w + l*l)}" />
