Commit message: Create tall block URDF model

File: block_tall.urdf (robot description, URDF)
Before this commit: robot pusher, 1 links, 0 joints
Links:
- link base_link: mass 1.0 -> 1; geometry collision box size=0.2 0.2 0.15; visual box size=0.2 0.2 0.15

File: models/_square_base.xacro (robot description, xacro)
@@ -1,13 +1,13 @@
 <?xml version="1.0"?>
-<robot name="wall" xmlns:xacro="http://www.ros.org/wiki/xacro">
-<xacro:macro name="wall" params="w l h">
-<xacro:property name="m" value="10" />
-<xacro:property name="Ih" value="${1/12*m*(w*w + l*l)}" />
-<xacro:property name="Iw" value="${1/12*m*(h*h + l*l)}" />
-<xacro:property name="Il" value="${1/12*m*(w*w + h*h)}" />
+<robot name="square" xmlns:xacro="http://www.ros.org/wiki/xacro">
+<xacro:macro name="square" params="s h m">
+<xacro:property name="Ih" value="${1/12*m*(s*s + s*s)}" />
+<xacro:property name="Iw" value="${1/12*m*(h*h + s*s)}" />
+<xacro:property name="Il" value="${1/12*m*(s*s + h*h)}" />
   <link name="base_link">
     <contact>
-      <lateral_friction value="0.7"/>
-      <spinning_friction value=".001"/>
+      <lateral_friction value="0.8"/>
+      <spinning_friction value=".05"/>
+      <rolling_friction value=".01"/>
     </contact>
     <inertial>
@@ -19,8 +19,8 @@
       <origin rpy="0 0 0" xyz="0.0 0.0 0.0"/>
       <geometry>
-        <box size="${l} ${w} ${h}"/>
+        <box size="${s} ${s} ${h}"/>
       </geometry>
       <material name="blockmat">
-        <color rgba="0.5 0.5 0.5 0.8"/>
+        <color rgba="0.1 0.7 0.1 0.8"/>
       </material>
     </visual>
@@ -28,5 +28,5 @@
       <origin rpy="0 0 0" xyz="0.0 0.0 0.0"/>
       <geometry>
-        <box size="${l} ${w} ${h}"/>
+        <box size="${s} ${s} ${h}"/>
       </geometry>
     </collision>

File: models/block_big.xacro (robot description, xacro)
@@ -1,37 +1,5 @@
 <?xml version="1.0"?>
 <robot xmlns:xacro="http://www.ros.org/wiki/xacro" name="block_big">
-<xacro:property name="m" value="3.0" />
-<xacro:property name="l" value="0.30" />
-<xacro:property name="w" value="0.30" />
-<xacro:property name="h" value="0.05" />
-<xacro:property name="Ih" value="${1/12*m*(w*w + l*l)}" />
-<xacro:property name="Iw" value="${1/12*m*(h*h + l*l)}" />
-<xacro:property name="Il" value="${1/12*m*(w*w + h*h)}" />
-  <link name="base_link">
-    <contact>
-      <lateral_friction value="0.8"/>
-      <spinning_friction value=".05"/>
-      <rolling_friction value=".01"/>
-    </contact>
-    <inertial>
-      <origin rpy="0 0 0" xyz="0 0 0"/>
-      <mass value="${m}"/>
-      <inertia ixx="${Il}" ixy="0" ixz="0" iyy="${Iw}" iyz="0" izz="${Ih}"/>
-    </inertial>
-    <visual>
-      <origin rpy="0 0 0" xyz="0.0 0.0 0.0"/>
-      <geometry>
-        <box size="${l} ${w} ${h}"/>
-      </geometry>
-      <material name="blockmat">
-        <color rgba="0.1 0.7 0.1 0.8"/>
-      </material>
-    </visual>
-    <collision>
-      <origin rpy="0 0 0" xyz="0.0 0.0 0.0"/>
-      <geometry>
-        <box size="${l} ${w} ${h}"/>
-      </geometry>
-    </collision>
- </link>
+<xacro:include filename="_square_base.xacro"/>
+<square s="0.3" h="0.05" m="3.0"/>
 </robot>
