Commit message: Fix collision radius of cylinder to match visual radius

File: topple_cylinder.urdf (robot description, URDF)
Before this commit: robot topple_cylinder, 1 links, 0 joints
Links:
- link base_link: geometry collision cylinder length=0.25 radius=0.12; visual cylinder length=0.25 radius=0.12
